Commit message: remove biases/ remove Gazebo pkg / move all models in simulator_pkg_models

File: simulator_pkg_models/simple_camera_model.xacro (robot description, xacro)
@@ -7,5 +7,6 @@
       <parent link="world"/>
       <child link="camera_link"/>
-      <origin rpy="0.0 1.5708 1.5708" xyz="0 0.0 0.5"/>
+      <!--<origin rpy="0.0 1.5708 1.5708" xyz="0 0.0 0.5"/>-->
+      <origin rpy="0.0 0.0 0.0" xyz="0 0.0 0.0"/>
   </joint>
   <link name="camera_link">

Commit message: make the camera model a floating object

File: simulator_pkg_models/simple_camera_model.xacro (robot description, xacro)
@@ -4,5 +4,5 @@
       <origin xyz="0.0 0.0 0.0"/>
   </link>
-  <joint name="camera_joint" type="fixed">
+  <joint name="camera_joint" type="floating">
       <parent link="world"/>
       <child link="camera_link"/>
